File: Battery Top/Battery Top/Battery Top.kicad_sch (KiCad schematic)
At the start: 6 parts, among them J1 JST_PWR_CON, J2 VBAT+_2, J3 VBAT+_1, J4 GND_R, J6 GND_L

Commit message: fixed footprint for fuse
Parts:
- F1: footprint Fuse:Fuse_1206_3216Metric -> Capacitor_SMD:C_1812_4532Metric
Changed lines of the file:
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@@
 			)
 		)
-		(property "Footprint" "Fuse:Fuse_1206_3216Metric"
+		(property "Footprint" "Capacitor_SMD:C_1812_4532Metric"
 			(at 135.89 140.97 0)
 			(hide yes)
