File: Battery Top/Kicad/Battery Top.kicad_sch (KiCad schematic)
At the start: 6 parts, among them J1 JST_PWR_CON, J2 VBAT+_2, J3 VBAT+_1, J4 GND_R, J6 GND_L

Commit message: Add required mechanical parts to README; update fuse footprint
- README: add "Additional parts required (beyond the BOMs)" section
  (battery, O-ring, stainless print, battery tabs, pogo pins)
- Battery Top: change fuse footprint
- Remove leftover stray Battery Top.kicad_pro from restructure

Co-Authored-By: Claude Opus 4.8 <noreply@anthropic.com>
Parts:
- added J5: DATA_1, Radio Library:Pogo Battery 7MM, symbol Connector:Conn_01x01_Pin
Connections:
- net DATA: now also J5.1 (Pin_1)
Changed lines of the file:
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@@
+		)
+	)
+	(label "DATA"
+		(at 157.48 107.95 180)
+		(effects
+			(font
+				(size 1.27 1.27)
+			)
+			(justify right bottom)
 		)
 	)
@@
 					(unit 1)
 				)
+			)
+		)
+	)
+	(symbol
+		(lib_id "Connector:Conn_01x01_Pin")
+		(at 162.56 107.95 180)
+		(unit 1)
+		(body_style 1)
+		(exclude_from_sim no)
+		(in_bom yes)
+		(on_board yes)
+		(in_pos_files yes)
+		(dnp no)
+		(property "Reference" "J5"
+			(at 161.925 68.58 0)
+			(hide yes)
+			(show_name no)
+			(do_not_autoplace no)
+			(effects
+				(font
+					(size 1.27 1.27)
+				)
+			)
+		)
+		(property "Value" "DATA_1"
+			(at 161.925 110.49 0)
+			(show_name no)
+			(do_not_autoplace no)
+			(effects
+				(font
+					(size 1.27 1.27)
+				)
+			)
+		)
+		(property "Footprint" "Radio Library:Pogo Battery 7MM"
+			(at 162.56 107.95 0)
+			(hide yes)
+			(show_name no)
+			(do_not_autoplace no)
+			(effects
+				(font
+					(size 1.27 1.27)
+				)
+			)
+		)
+		(property "Datasheet" ""
+			(at 162.56 107.95 0)
+			(hide yes)
+			(show_name no)
+			(do_not_autoplace no)
+			(effects
+				(font
+					(size 1.27 1.27)
+				)
+			)
+		)
+		(property "Description" "Generic connector, single row, 01x01, script generated"
+			(at 162.56 107.95 0)
+			(hide yes)
+			(show_name no)
+			(do_not_autoplace no)
+			(effects
+				(font
+					(size 1.27 1.27)
+				)
+			)
+		)
+		(pin "1"
+		)
+		(instances
+			(project "Battery Top"
+				(path "/4d066849-3f37-4480-bd30-0688a5a62bf8"
+					(reference "J5")
+					(unit 1)
+				)
