File: Battery Top/Kicad/Battery Top.kicad_pcb (KiCad board)
At the start: 2 copper layers, 64 x 21 mm, 7 parts, among them J1 JST_PWR_CON, J2 VBAT+_2, J3 VBAT+_1, J4 GND_R, J5 DATA_1, J6 GND_L

Commit message: footprint
Parts:
- F1: footprint Capacitor_SMD:C_1812_4532Metric -> Resistor_SMD:R_1812_4532Metric
Changed lines of the file:
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@@
 		)
 	)
-	(footprint "Capacitor_SMD:C_1812_4532Metric"
+	(footprint "Resistor_SMD:R_1812_4532Metric"
 		(layer "F.Cu")
 		(at 157 99 180)
-		(descr "Capacitor SMD 1812 (4532 Metric), square (rectangular) end terminal, IPC-7351 nominal, (Body size source: IPC-SM-782 page 76, https://www.pcb-3d.com/wordpress/wp-content/uploads/ipc-sm-782a_amendment_1_and_2.pdf)")
-		(tags "capacitor")
+		(descr "Resistor SMD 1812 (4532 Metric), square (rectangular) end terminal, IPC-7351 nominal, (Body size source: https://www.nikhef.nl/pub/departments/mt/projects/detectorR_D/dtddice/ERJ2G.pdf)")
+		(tags "resistor")
 		(property "Reference" "F1"
 			(at 0 -2.65 180)
@@
 		(duplicate_pad_numbers_are_jumpers no)
 		(fp_line
-			(start -1.161252 1.71)
-			(end 1.161252 1.71)
+			(start -1.386252 1.71)
+			(end 1.386252 1.71)
 			(stroke
 				(width 0.12)
@@
 		)
 		(fp_line
-			(start -1.161252 -1.71)
-			(end 1.161252 -1.71)
+			(start -1.386252 -1.71)
+			(end 1.386252 -1.71)
 			(stroke
 				(width 0.12)
@@
 		)
 		(fp_rect
-			(start -3 -1.95)
-			(end 3 1.95)
+			(start -2.95 -1.95)
+			(end 2.95 1.95)
 			(stroke
 				(width 0.05)
@@
 		)
 		(pad "1" smd roundrect
-			(at -2.05 0 180)
-			(size 1.4 3.4)
+			(at -2.1375 0 180)
+			(size 1.125 3.4)
 			(layers "F.Cu" "F.Mask" "F.Paste")
-			(roundrect_rratio 0.178571)
+			(roundrect_rratio 0.222222)
 			(net "/VBAT+")
 			(pintype "passive")
 		)
 		(pad "2" smd roundrect
-			(at 2.05 0 180)
-			(size 1.4 3.4)
+			(at 2.1375 0 180)
+			(size 1.125 3.4)
 			(layers "F.Cu" "F.Mask" "F.Paste")
-			(roundrect_rratio 0.178571)
+			(roundrect_rratio 0.222222)
 			(net "/VBAT+_P")
 			(pintype "passive")
 		)
 		(embedded_fonts no)
-		(model "${KICAD10_3DMODEL_DIR}/Capacitor_SMD.3dshapes/C_1812_4532Metric.step"
+		(model "${KICAD10_3DMODEL_DIR}/Resistor_SMD.3dshapes/R_1812_4532Metric.step"
 			(offset
 				(xyz 0 0 0)
@@
 	(footprint "Radio Library:Pogo Battery 7MM"
 		(layer "F.Cu")
+		(at 151 100)
+		(property "Reference" "J5"
+			(at 0 -0.5 0)
+			(unlocked yes)
+			(layer "F.SilkS")
+			(hide yes)
+			(effects
+				(font
+					(size 1 1)
+					(thickness 0.1)
+				)
+			)
+		)
+		(property "Value" "DATA_1"
+			(at 0 3 0)
+			(unlocked yes)
+			(layer "F.Fab")
+			(hide yes)
+			(effects
+				(font
+					(size 1 1)
+					(thickness 0.15)
+				)
+			)
+		)
+		(property "Datasheet" ""
+			(at 0 0 0)
+			(unlocked yes)
+			(layer "F.Fab")
+			(hide yes)
+			(effects
+				(font
+					(size 1 1)
+					(thickness 0.15)
+				)
+			)
+		)
+		(property "Description" "Generic connector, single row, 01x01, script generated"
+			(at 0 0 0)
+			(unlocked yes)
+			(layer "F.Fab")
+			(hide yes)
+			(effects
+				(font
+					(size 1 1)
+					(thickness 0.15)
+				)
+			)
+		)
+		(property ki_fp_filters "Connector*:*_1x??_*")
+		(sheetname "/")
+		(sheetfile "Battery Top.kicad_sch")
+		(units
+			(unit
+				(name "A")
+				(pins "1")
+			)
+		)
+		(attr smd)
+		(duplicate_pad_numbers_are_jumpers no)
+		(pad "1" thru_hole circle
+			(at 0 0)
+			(size 2.5 2.5)
+			(drill 1.6)
+			(layers "*.Cu" "*.Mask")
+			(remove_unused_layers no)
+			(net "/DATA")
+			(pinfunction "Pin_1_1")
+			(pintype "passive")
+			(thermal_bridge_angle 90)
+		)
+		(embedded_fonts no)
+	)
+	(footprint "Radio Library:Pogo Battery 7MM"
+		(layer "F.Cu")
 		(at 151 104)
 		(property "Reference" "J2"
@@
 		(embedded_fonts no)
 	)
-	(footprint "Radio Library:Pogo Battery 7MM"
-		(layer "F.Cu")
-		(at 151 100)
-		(property "Reference" "J5"
-			(at 0 -0.5 0)
-			(unlocked yes)
-			(layer "F.SilkS")
-			(hide yes)
-			(effects
-				(font
-					(size 1 1)
-					(thickness 0.1)
-				)
-			)
-		)
-		(property "Value" "DATA_1"
-			(at 0 3 0)
-			(unlocked yes)
-			(layer "F.Fab")
-			(hide yes)
-			(effects
-				(font
-					(size 1 1)
-					(thickness 0.15)
-				)
-			)
-		)
-		(property "Datasheet" ""
-			(at 0 0 0)
-			(unlocked yes)
-			(layer "F.Fab")
-			(hide yes)
-			(effects
-				(font
-					(size 1 1)
-					(thickness 0.15)
-				)
-			)
-		)
-		(property "Description" "Generic connector, single row, 01x01, script generated"
-			(at 0 0 0)
-			(unlocked yes)
-			(layer "F.Fab")
-			(hide yes)
-			(effects
-				(font
-					(size 1 1)
-					(thickness 0.15)
-				)
-			)
-		)
-		(property ki_fp_filters "Connector*:*_1x??_*")
-		(sheetname "/")
-		(sheetfile "Battery Top.kicad_sch")
-		(units
-			(unit
-				(name "A")
-				(pins "1")
-			)
-		)
-		(attr smd)
-		(duplicate_pad_numbers_are_jumpers no)
-		(pad "1" thru_hole circle
-			(at 0 0)
-			(size 2.5 2.5)
-			(drill 1.6)
-			(layers "*.Cu" "*.Mask")
-			(remove_unused_layers no)
-			(net "/DATA")
-			(pinfunction "Pin_1_1")
-			(pintype "passive")
-			(thermal_bridge_angle 90)
-		)
-		(embedded_fonts no)
-	)
 	(footprint "Radio Library:Bolt Pad 4.25"
 		(layer "F.Cu")
@@
 	)
 	(segment
+		(start 151 100)
+		(end 150.5 100.5)
+		(width 0.5)
+		(layer "F.Cu")
+		(net "/DATA")
+	)
+	(segment
 		(start 136.5 100.5)
 		(end 137 100.5)
@@
 		(layer "F.Cu")
 		(net "/DATA")
-	)
-	(segment
-		(start 151 100)
-		(end 150.5 100.5)
-		(width 0.5)
-		(layer "F.Cu")
-		(net "/DATA")
