File: Battery Cell Holder/Battery Cell Holder Top PCB/Kicad/Battery Cell Holder Top PCB.kicad_pcb (KiCad board)
At the start: 2 copper layers, 39 x 70 mm, 10 parts

Commit message: fixes to boards
Parts:
- 12.6V: renamed from C1; moved to B.Cu
- 12.6V: renamed from BT1; footprint BatterySpringContact:Keystone_5222_SpringContact_THM -> C19724688:TH-2_BD10.0_F10-12-0.5-1.3UU-SUS304; moved to B.Cu
- 12.6V: renamed from BT2; footprint BatterySpringContact:Keystone_5222_SpringContact_THM -> C19724688:TH-2_BD10.0_F10-12-0.5-1.3UU-SUS304; moved to B.Cu
- 4.2V: renamed from BT5; footprint BatterySpringContact:Keystone_5222_SpringContact_THM -> C19724688:TH-2_BD10.0_F10-12-0.5-1.3UU-SUS304; moved to B.Cu
- 4.2V: renamed from BT6; footprint BatterySpringContact:Keystone_5222_SpringContact_THM -> C19724688:TH-2_BD10.0_F10-12-0.5-1.3UU-SUS304; moved to B.Cu
- 8.4V: renamed from BT3; footprint BatterySpringContact:Keystone_5222_SpringContact_THM -> C19724688:TH-2_BD10.0_F10-12-0.5-1.3UU-SUS304; moved to B.Cu
- 8.4V: renamed from BT4; footprint BatterySpringContact:Keystone_5222_SpringContact_THM -> C19724688:TH-2_BD10.0_F10-12-0.5-1.3UU-SUS304; moved to B.Cu
- turned 12.6V to 180 degrees (x3)
- turned 4.2V to 180 degrees (x2)
- turned 8.4V to 180 degrees (x2)
- renumbered C1 to 12.6V, C3 to 8.4V
Connections:
- 12.6V pad 1: /C1 -> /C3 (x4)
- 4.2V pad 1: /C3 -> /C2 (x2)
- 8.4V pad 1: /C3 -> /C2 (x2)
- 8.4V pad 1: /C1 -> /C2 (x2)
Routing:
- net /C2: track 0.00 -> 104.6 mm
- net /C1: track 103.4 -> 0.00 mm
- net /C3: track 50.1 -> 51.0 mm
Other:
- board text added: "+"
- board text added: "-"
- board text added: "12.6V"
- board text added: "4.2V"
- board text added: "TOP PANEL [UNDER SIDE]"
- board text removed: "TOP PANEL [UNDERSIDE]"

Commit message: fixed
Parts:
- renumbered 12.6V to BT1, 12.6V to BT2, 8.4V to BT3, 8.4V to BT4, 4.2V to BT5, 4.2V to BT6, 12.6V to TP1, 12.6V to TP2, 8.4V to TP3, 8.4V to TP4
Changed lines of the file:
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@@
 		(descr "Soldered wire connection, for a single 1.5 mm² wire, reinforced insulation, conductor diameter 1.7mm, outer diameter 3.9mm, size source Multi-Contact FLEXI-xV 1.5 (https://www.staubli.com/content/dam/ecs/catalogs-brochures/TM/CAB-Main-11014119-en.pdf#page=11), bend radius 3 times outer diameter")
 		(tags "connector wire 1.5sqmm")
-		(property "Reference" "12.6V"
+		(property "Reference" "TP2"
 			(at 0 -3.15 0)
 			(layer "B.SilkS")
@@
 		(property ki_fp_filters "Pin* Test*")
 		(sheetname "/")
-		(sheetfile "Battery Cell Bottom PCB.kicad_sch")
+		(sheetfile "Battery Cell Holder Top PCB.kicad_sch")
 		(units
 			(unit
@@
 		(descr "Soldered wire connection, for a single 1.5 mm² wire, reinforced insulation, conductor diameter 1.7mm, outer diameter 3.9mm, size source Multi-Contact FLEXI-xV 1.5 (https://www.staubli.com/content/dam/ecs/catalogs-brochures/TM/CAB-Main-11014119-en.pdf#page=11), bend radius 3 times outer diameter")
 		(tags "connector wire 1.5sqmm")
-		(property "Reference" "8.4V"
+		(property "Reference" "TP4"
 			(at 0 -3.15 0)
 			(layer "B.SilkS")
@@
 		(property ki_fp_filters "Pin* Test*")
 		(sheetname "/")
-		(sheetfile "Battery Cell Bottom PCB.kicad_sch")
+		(sheetfile "Battery Cell Holder Top PCB.kicad_sch")
 		(units
 			(unit
@@
 		(descr "Soldered wire connection, for a single 1.5 mm² wire, reinforced insulation, conductor diameter 1.7mm, outer diameter 3.9mm, size source Multi-Contact FLEXI-xV 1.5 (https://www.staubli.com/content/dam/ecs/catalogs-brochures/TM/CAB-Main-11014119-en.pdf#page=11), bend radius 3 times outer diameter")
 		(tags "connector wire 1.5sqmm")
-		(property "Reference" "8.4V"
+		(property "Reference" "TP3"
 			(at 0 -3.15 0)
 			(layer "B.SilkS")
@@
 		(property ki_fp_filters "Pin* Test*")
 		(sheetname "/")
-		(sheetfile "Battery Cell Bottom PCB.kicad_sch")
+		(sheetfile "Battery Cell Holder Top PCB.kicad_sch")
 		(units
 			(unit
@@
 		(descr "Soldered wire connection, for a single 1.5 mm² wire, reinforced insulation, conductor diameter 1.7mm, outer diameter 3.9mm, size source Multi-Contact FLEXI-xV 1.5 (https://www.staubli.com/content/dam/ecs/catalogs-brochures/TM/CAB-Main-11014119-en.pdf#page=11), bend radius 3 times outer diameter")
 		(tags "connector wire 1.5sqmm")
-		(property "Reference" "12.6V"
+		(property "Reference" "TP1"
 			(at 0 3.15 0)
 			(layer "B.SilkS")
@@
 		(property ki_fp_filters "Pin* Test*")
 		(sheetname "/")
-		(sheetfile "Battery Cell Bottom PCB.kicad_sch")
+		(sheetfile "Battery Cell Holder Top PCB.kicad_sch")
 		(units
 			(unit
@@
 		(layer "B.Cu")
 		(at 97.187074 84.78834 180)
-		(property "Reference" "12.6V"
+		(property "Reference" "BT1"
 			(at 0 4 0)
 			(layer "B.SilkS")
@@
 				(font
 					(size 1.27 1.27)
+					(thickness 0.15)
 				)
 				(justify mirror)
@@
 		)
 		(sheetname "/")
-		(sheetfile "Battery Cell Bottom PCB.kicad_sch")
+		(sheetfile "Battery Cell Holder Top PCB.kicad_sch")
 		(units
 			(unit
@@
 		(layer "B.Cu")
 		(at 97.187074 103.78834 180)
-		(property "Reference" "8.4V"
+		(property "Reference" "BT3"
 			(at 0 4 0)
 			(layer "B.SilkS")
@@
 				(font
 					(size 1.27 1.27)
+					(thickness 0.15)
 				)
 				(justify mirror)
@@
 		)
 		(sheetname "/")
-		(sheetfile "Battery Cell Bottom PCB.kicad_sch")
+		(sheetfile "Battery Cell Holder Top PCB.kicad_sch")
 		(units
 			(unit
@@
 		(layer "B.Cu")
 		(at 114.216932 75.309426 180)
-		(property "Reference" "12.6V"
+		(property "Reference" "BT2"
 			(at 0 4 0)
 			(layer "B.SilkS")
@@
 				(font
 					(size 1.27 1.27)
+					(thickness 0.15)
 				)
 				(justify mirror)
@@
 		)
 		(sheetname "/")
-		(sheetfile "Battery Cell Bottom PCB.kicad_sch")
+		(sheetfile "Battery Cell Holder Top PCB.kicad_sch")
 		(units
 			(unit
@@
 		(layer "B.Cu")
 		(at 114.216932 94.309426 180)
-		(property "Reference" "8.4V"
+		(property "Reference" "BT4"
 			(at 0 4 0)
 			(layer "B.SilkS")
@@
 				(font
 					(size 1.27 1.27)
+					(thickness 0.15)
 				)
 				(justify mirror)
@@
 		)
 		(sheetname "/")
-		(sheetfile "Battery Cell Bottom PCB.kicad_sch")
+		(sheetfile "Battery Cell Holder Top PCB.kicad_sch")
 		(units
 			(unit
@@
 		(layer "B.Cu")
 		(at 97.187074 122.78834 180)
-		(property "Reference" "4.2V"
+		(property "Reference" "BT5"
 			(at 0 4 0)
 			(layer "B.SilkS")
@@
 				(font
 					(size 1.27 1.27)
+					(thickness 0.15)
 				)
 				(justify mirror)
@@
 		)
 		(sheetname "/")
-		(sheetfile "Battery Cell Bottom PCB.kicad_sch")
+		(sheetfile "Battery Cell Holder Top PCB.kicad_sch")
 		(units
 			(unit
@@
 		(layer "B.Cu")
 		(at 114.216932 113.309426 180)
-		(property "Reference" "4.2V"
+		(property "Reference" "BT6"
 			(at 0 4 0)
 			(layer "B.SilkS")
@@
 				(font
 					(size 1.27 1.27)
+					(thickness 0.15)
 				)
 				(justify mirror)
@@
 		)
 		(sheetname "/")
-		(sheetfile "Battery Cell Bottom PCB.kicad_sch")
+		(sheetfile "Battery Cell Holder Top PCB.kicad_sch")
 		(units
 			(unit
